Commit message: fix(sim): Added explicitely defined ground plane to world file. Sim was having trouble reachout out to gazebo repo. Should really migrate to newer version of gazebo soon.

File: turtle_ws/src/turtlebot_nav_control/urdf/turtlebot_nav_control.urdf.xacro (robot description, xacro)
@@ -51,5 +51,5 @@
     </visual>
     <collision>
-      <origin xyz="-0.032 0 0.070" rpy="0 0 0"/>
+      <origin xyz="-0.032 0 0.0715" rpy="0 0 0"/>
       <geometry>
         <box size="0.140 0.140 0.143"/>
